File: hardware/FCom-8.kicad_pcb (KiCad board)
At the start: 2 copper layers, 94 x 127 mm, 74 parts, among them J201 4090 USB-C, J202 9V battery, SW101 SW_DIP_x08, SW102 SW_DIP_x08, SW104 SW_DIP_x04, SW105 G19AP, SW301 Q/1/STOP, SW302 W/2/CH0, SW303 E/3/CH1, SW304 R/4/CH2, SW305 T/5/CH3, SW306 Y/6/_, SW307 U/7/-, SW308 I/8/+, SW309 O/9/=, SW310 P/0, SW311 A/!/`, SW312 S/"/CH4, SW313 D/$/CH5, SW314 F/%/CH6, SW315 G/^/CH7, SW316 H/&/{, SW317 J/*/}, SW318 K/(/[, SW319 L/)/], SW320 BKSP/DEL, SW321 SHIFT, SW322 Z/\/|, SW323 X/;/:, SW324 C/'/@, SW325 V/#/~, SW326 B/,/<, SW327 N/./>, SW328 M///?, SW329 SYM, SW330 SPC/ENT, U101 65C02, U102 AS6C1008-55PCN, U103 65C22, U104 74LS04, U105 74LS08, U106 74LS21, U201 LM1117T-5.0, U301 MCP23S17_SP, U302 NHD-0420DZ-FL-YBW

Commit message: Add final planned components
Parts:
- added D102: Green LED, LED_THT:LED_D5.0mm, F.Cu at (124.5, 104.1)
- added D103: Red LED, LED_THT:LED_D5.0mm, F.Cu at (139.7, 104.1)
- added D104: Blue LED, LED_THT:LED_D5.0mm, F.Cu at (61.0, 88.9)
- added D204: Red LED, LED_THT:LED_D5.0mm, F.Cu at (116.8, 27.9)
- added J101: Conn_01x04, Connector_PinHeader_2.54mm:PinHeader_1x04_P2.54mm_Vertical, F.Cu at (142.2, 55.9)
- added R107: 330, Resistor_THT:R_Axial_DIN0207_L6.3mm_D2.5mm_P7.62mm_Horizontal, F.Cu at (142.2, 121.9)
- added R108: 330, Resistor_THT:R_Axial_DIN0207_L6.3mm_D2.5mm_P7.62mm_Horizontal, F.Cu at (104.1, 109.2)
- added R109: 330, Resistor_THT:R_Axial_DIN0207_L6.3mm_D2.5mm_P7.62mm_Horizontal, F.Cu at (53.3, 121.9)
- added R201: 100k, Resistor_THT:R_Axial_DIN0207_L6.3mm_D2.5mm_P7.62mm_Horizontal, F.Cu at (114.3, 55.9)
- added R202: 47k, Resistor_THT:R_Axial_DIN0207_L6.3mm_D2.5mm_P7.62mm_Horizontal, F.Cu at (124.5, 58.8)
- added R203: 330, Resistor_THT:R_Axial_DIN0207_L6.3mm_D2.5mm_P7.62mm_Horizontal, F.Cu at (119.4, 33.0)
- added Y101: ECS-100AX-010, Components:ECS-100AX-010, F.Cu at (101.6, 119.4)
- SW105: footprint Connector_PinHeader_2.54mm:PinHeader_1x03_P2.54mm_Vertical -> Components:G19AP
- U101: value 65C02 -> W65C02S6TPG-14
- U103: value 65C22 -> W65C22N6TPG-14
- moved G*** 12.7 mm to (66.0, 113.0)
- moved R102 5.08 mm to (53.3, 94.0)
- moved SW105 3.80 mm to (129.5, 99.1), turned to 0 degrees
- moved C206 2.54 mm to (106.7, 88.9)
Connections:
- RN103 pad 2: /A15 -> /A12
- RN103 pad 3: /A14 -> /A13
- RN103 pad 4: /A13 -> /A14
- RN103 pad 5: /A12 -> /A15
- SW104 pad 2: unconnected-(SW104-Pad2) -> VCC
- SW104 pad 3: unconnected-(SW104-Pad3) -> GND
- SW104 pad 4: unconnected-(SW104-Pad4) -> GND
- SW104 pad 5: unconnected-(SW104-Pad5) -> KB_SWB
- SW104 pad 6: unconnected-(SW104-Pad6) -> KB_SWA
- SW104 pad 7: unconnected-(SW104-Pad7) -> DISP_BL
- U102 pad 13: /D0 -> /D2
- U102 pad 15: /D2 -> /D0
- U102 pad 2: RAM_BANKSEL -> /A10
- U102 pad 23: /A10 -> RAM_BANKSEL
- U102 pad 25: /A11 -> /A15
- U102 pad 26: /A9 -> /A14
- U102 pad 27: /A8 -> /A13
- U102 pad 28: /A13 -> /A12
- U102 pad 3: /A14 -> /A9
- U102 pad 31: /A15 -> /A11
- U102 pad 4: /A12 -> /A8
- U103 pad 10: KB_SO -> Net-(U103-PB0)
- U103 pad 11: KB_SI -> DISP_RS
- U103 pad 12: KB_SCK -> DISP_RW
- U103 pad 13: ~{KB_CS} -> DISP_E
- U103 pad 14: unconnected-(U103-PB4-Pad14) -> KB_SO
- U103 pad 15: unconnected-(U103-PB5-Pad15) -> KB_SI
- U103 pad 16: unconnected-(U103-PB6-Pad16) -> KB_SCK
- U103 pad 17: unconnected-(U103-PB7-Pad17) -> ~{KB_CS}
- U103 pad 18: unconnected-(U103-CB1-Pad18) -> Net-(J101-Pin_3)
- U103 pad 19: unconnected-(U103-CB2-Pad19) -> Net-(J101-Pin_2)
- U103 pad 39: unconnected-(U103-CA2-Pad39) -> ~{BATLOW}
- U106 pad 12: /A14 -> /A15
- U106 pad 13: /A15 -> /A14
- U301 pad 1: unconnected-(U301-GPB0-Pad1) -> KB_SWA
- U301 pad 2: unconnected-(U301-GPB1-Pad2) -> KB_SWB
- U302 pad 15: VCC -> DISP_BL
