File: hardware/FCom-8.kicad_sch (KiCad schematic)
At the start: 21 parts, among them SW101 SW_DIP_x08, SW102 SW_DIP_x08, SW104 SW_DIP_x04, SW105 G19AP, U101 65C02, U102 AS6C1008-55PCN, U103 65C22, U104 74LS04, U105 74LS08, U106 74LS21

Commit message: Add final planned components
Parts:
- added D102: Green LED, LED_THT:LED_D5.0mm, symbol Device:LED
- added D103: Red LED, LED_THT:LED_D5.0mm, symbol Device:LED
- added D104: Blue LED, LED_THT:LED_D5.0mm, symbol Device:LED
- added J101: Conn_01x04, Connector_PinHeader_2.54mm:PinHeader_1x04_P2.54mm_Vertical, symbol Connector_Generic:Conn_01x04
- added R107, R108, R109: 330, Resistor_THT:R_Axial_DIN0207_L6.3mm_D2.5mm_P7.62mm_Horizontal, symbol Device:R
- added Y101: ECS-100AX-010, Components:ECS-100AX-010, symbol Components:ECS-100AX-010
- SW105: footprint Connector_PinHeader_2.54mm:PinHeader_1x03_P2.54mm_Vertical -> Components:G19AP
- U101: value 65C02 -> W65C02S6TPG-14
- U103: value 65C22 -> W65C22N6TPG-14
Connections:
- net A10: now also U102.2 (A16); no longer U102.23 (A10)
- net A11: now also U102.31 (A15); no longer U102.25 (A11)
- net A12: now also RN103.2 (R1), U102.28 (A13); no longer RN103.5 (R4), U102.4 (A12)
- net A13: now also RN103.3 (R2), U102.27 (A8); no longer RN103.4 (R3), U102.28 (A13)
- net A14: now also RN103.4 (R3), U102.26 (A9), U106.13; no longer RN103.3 (R2), U102.3 (A14), U106.12
- net A15: now also RN103.5 (R4), U102.25 (A11), U106.12; no longer RN103.2 (R1), U102.31 (A15), U106.13
- net A8: now also U102.4 (A12); no longer U102.27 (A8)
- net A9: now also U102.3 (A14); no longer U102.26 (A9)
- net CLOCK: now also Y101.8 (OUT)
- net D0: now also U102.15 (DQ2); no longer U102.13 (DQ0)
- net D2: now also U102.13 (DQ0); no longer U102.15 (DQ2)
- net GND: now also SW104.3, SW104.4, D102.1 (K), D103.1 (K), D104.1 (K), J101.1 (Pin_1), Y101.7 (GND)
- net KB_SCK: now also U103.16 (PB6); no longer U103.12 (PB2)
- net KB_SI: now also U103.15 (PB5); no longer U103.11 (PB1)
- net KB_SO: now also U103.14 (PB4); no longer U103.10 (PB0)
- net RAM_BANKSEL: now also U102.23 (A10); no longer U102.2 (A16)
- net VBS: now also R107.1
- net VCC: now also SW104.2, J101.4 (Pin_4), R108.2, Y101.14 (+5V)
- net ~{KB_CS}: now also U103.17 (PB7); no longer U103.13 (PB3)
- net at U103.18 (CB1): now also J101.3 (Pin_3)
- net at U103.19 (CB2): now also J101.2 (Pin_2)
- net ~{BATLOW}: now reaches U103.39 (CA2)
- net KB_SWB: now reaches SW104.5
- net KB_SWA: now reaches SW104.6
- net DISP_BL: now reaches SW104.7
- new net: D102.2 (A), R107.2
- new net: R109.2, U103.10 (PB0)
- new net: D103.2 (A), R108.1
- new net: D104.2 (A), R109.1
- new net DISP_E: U103.13 (PB3)
- new net DISP_RS: U103.11 (PB1)
- new net DISP_RW: U103.12 (PB2)
Other:
- note added: "Backlight switch"
- note added: "Bootstrap high-byte address ($FFxx)"
- note added: "CPU power LED"
- note added: "Crystal oscillator"
- note added: "Custom LED"
- note added: "Custom switch A"
- note added: "Custom switch B"
- note added: "Logical pins reassigned for ease of routing"
- note added: "RAM write confirmatory LED"
- note added: "Serial comms header"
- moved on the sheet: C101, D101, R101, R102, R103, R104, R105, R106, RN101, RN102, RN103, SW101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
