File: hardware/Aletheia.kicad_pcb (KiCad board)
At the start: 12 copper layers, 94 x 127 mm, 85 parts, among them J101 Conn_01x04, J201 4090 USB-C, J202 9V battery, SW101 SW_DIP_x08, SW102 SW_DIP_x08, SW104 SW_DIP_x04, SW105 G19AP, SW301 Q/1/STOP, SW302 W/2/CH0, SW303 E/3/CH1, SW304 R/4/CH2, SW305 T/5/CH3, SW306 Y/6/_, SW307 U/7/-, SW308 I/8/+, SW309 O/9/=, SW310 P/0, SW311 A/!/`, SW312 S/"/CH4, SW313 D/$/CH5, SW314 F/%/CH6, SW315 G/^/CH7, SW316 H/&/{, SW317 J/*/}, SW318 K/(/[, SW319 L/)/], SW320 BKSP/DEL, SW321 SHIFT, SW322 Z/\/|, SW323 X/;/:, SW324 C/'/@, SW325 V/#/~, SW326 B/,/<, SW327 N/./>, SW328 M///?, SW329 SYM, SW330 SPC/ENT, U101 W65C02S6TPG-14, U102 AS6C1008-55PCN, U103 W65C22N6TPG-14, U104 74LS04, U105 74LS08, U106 74LS21, U201 LP2954AIT/NOPB, U301 MCP23S17_SP, U302 NHD-0420DZ-NSW-BBW, Y101 ECS-100AX-010

Commit message: Fix missing trace wire in hardware
Routing:
- net VCC: track 507.9 -> 533.8 mm
Changed lines of the file:
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@@
+	)
+	(segment
+		(start 109.281 62.399)
+		(end 108.18 63.5)
+		(width 0.2)
+		(layer "In2.Cu")
+		(net 2)
 	)
 	(segment
@@
 	)
 	(segment
+		(start 127 73.66)
+		(end 125.10495 73.66)
+		(width 0.2)
+		(layer "In2.Cu")
+		(net 2)
+	)
+	(segment
 		(start 66.04 68.58)
 		(end 67.541 67.079)
@@
 	)
 	(segment
+		(start 117.21605 62.399)
+		(end 109.281 62.399)
+		(width 0.2)
+		(layer "In2.Cu")
+		(net 2)
+	)
+	(segment
 		(start 106.68 68.58)
 		(end 108.18 67.08)
@@
 	)
 	(segment
+		(start 120.481 69.03605)
+		(end 120.481 65.66395)
+		(width 0.2)
+		(layer "In2.Cu")
+		(net 2)
+	)
+	(segment
 		(start 99.06 81.28)
 		(end 106.68 73.66)
@@
 	)
 	(segment
+		(start 120.481 65.66395)
+		(end 117.21605 62.399)
+		(width 0.2)
+		(layer "In2.Cu")
+		(net 2)
+	)
+	(segment
 		(start 55.88 81.28)
 		(end 99.06 81.28)
@@
 		(width 0.2)
 		(layer "In2.Cu")
+		(net 2)
+	)
+	(segment
+		(start 125.10495 73.66)
+		(end 120.481 69.03605)
+		(width 0.2)
+		(layer "In2.Cu")
