File: hardware/Aletheia.kicad_pcb (KiCad board)
At the start: 12 copper layers, 94 x 127 mm, 85 parts, among them J101 Conn_01x04, J201 4090 USB-C, J202 9V battery, SW101 SW_DIP_x08, SW102 SW_DIP_x08, SW104 SW_DIP_x04, SW105 G19AP, SW301 Q/1/STOP, SW302 W/2/CH0, SW303 E/3/CH1, SW304 R/4/CH2, SW305 T/5/CH3, SW306 Y/6/_, SW307 U/7/-, SW308 I/8/+, SW309 O/9/=, SW310 P/0, SW311 A/!/`, SW312 S/"/CH4, SW313 D/$/CH5, SW314 F/%/CH6, SW315 G/^/CH7, SW316 H/&/{, SW317 J/*/}, SW318 K/(/[, SW319 L/)/], SW320 BKSP/DEL, SW321 SHIFT, SW322 Z/\/|, SW323 X/;/:, SW324 C/'/@, SW325 V/#/~, SW326 B/,/<, SW327 N/./>, SW328 M///?, SW329 SYM, SW330 SPC/ENT, U101 W65C02S6TPG-14, U102 AS6C1008-55PCN, U103 W65C22N6TPG-14, U104 74LS04, U105 74LS08, U106 74LS21, U201 LP2954AIT/NOPB, U301 MCP23S17_SP, U302 NHD-0420DZ-NSW-BBW, Y101 ECS-100AX-010

Commit message: Fix orientation of pins for mode switch in hardware
Connections:
- SW105 pad 4: VBS -> VCC
- SW105 pad 6: VCC -> VBS
Routing:
- net +5V: track 196.8 -> 194.9 mm
- net VBS: track 192.0 -> 190.5 mm
- net VCC: track 533.8 -> 533.1 mm
Changed lines of the file:
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@@
 			(layers "*.Cu" "*.Mask")
 			(remove_unused_layers no)
-			(net 40 "VBS")
+			(net 2 "VCC")
 			(pinfunction "4")
 			(pintype "passive")
@@
 			(layers "*.Cu" "*.Mask")
 			(remove_unused_layers no)
-			(net 40 "VBS")
+			(net 2 "VCC")
 			(pinfunction "4")
 			(pintype "passive")
@@
 			(layers "*.Cu" "*.Mask")
 			(remove_unused_layers no)
-			(net 2 "VCC")
+			(net 40 "VBS")
 			(pinfunction "6")
 			(pintype "passive")
@@
 			(layers "*.Cu" "*.Mask")
 			(remove_unused_layers no)
-			(net 2 "VCC")
+			(net 40 "VBS")
 			(pinfunction "6")
 			(pintype "passive")
@@
 	)
 	(segment
+		(start 134.62 99.06)
+		(end 134.62 101.6)
+		(width 1.5)
+		(layer "B.Cu")
+		(net 2)
+	)
+	(segment
 		(start 106.68 73.66)
 		(end 106.68 68.58)
@@
 	)
 	(segment
-		(start 129.54 99.06)
-		(end 129.54 101.6)
-		(width 1.5)
-		(layer "B.Cu")
-		(net 2)
-	)
-	(segment
 		(start 142.24 96.52)
 		(end 142.291 96.571)
@@
 	)
 	(segment
-		(start 75.799 40.239)
-		(end 98.659 40.239)
+		(start 127 99.06)
+		(end 128.407214 99.06)
 		(width 0.2)
 		(layer "In2.Cu")
@@
 	)
 	(segment
-		(start 128.27 72.39)
-		(end 127 73.66)
+		(start 75.799 40.239)
+		(end 98.659 40.239)
 		(width 0.2)
 		(layer "In2.Cu")
@@
 	)
 	(segment
-		(start 129.54 99.06)
-		(end 127 99.06)
+		(start 128.27 72.39)
+		(end 127 73.66)
 		(width 0.2)
 		(layer "In2.Cu")
@@
 	)
 	(segment
-		(start 134.550786 100.262)
-		(end 141.038 100.262)
+		(start 53.34 83.82)
+		(end 55.88 81.28)
 		(width 0.2)
 		(layer "In2.Cu")
@@
 	)
 	(segment
-		(start 53.34 83.82)
-		(end 55.88 81.28)
+		(start 55.88 68.58)
+		(end 58.42 66.04)
 		(width 0.2)
 		(layer "In2.Cu")
@@
 	)
 	(segment
-		(start 55.88 68.58)
-		(end 58.42 66.04)
+		(start 134.62 99.06)
+		(end 135.822 100.262)
 		(width 0.2)
 		(layer "In2.Cu")
@@
 	)
 	(segment
+		(start 133.819 102.401)
+		(end 134.62 101.6)
+		(width 0.2)
+		(layer "In2.Cu")
+		(net 2)
+	)
+	(segment
 		(start 67.479 31.919)
 		(end 68.58 33.02)
@@
 	)
 	(segment
+		(start 128.407214 99.06)
+		(end 131.748214 102.401)
+		(width 0.2)
+		(layer "In2.Cu")
+		(net 2)
+	)
+	(segment
 		(start 55.631057 37.499)
 		(end 54.441 38.689057)
@@
 	)
 	(segment
+		(start 131.748214 102.401)
+		(end 133.819 102.401)
+		(width 0.2)
+		(layer "In2.Cu")
+		(net 2)
+	)
+	(segment
 		(start 54.441 38.689057)
 		(end 54.441 52.239)
@@
 	)
 	(segment
-		(start 132.411786 102.401)
-		(end 134.550786 100.262)
-		(width 0.2)
-		(layer "In2.Cu")
-		(net 2)
-	)
-	(segment
 		(start 58.42 53.34)
 		(end 59.921 51.839)
@@
 	)
 	(segment
-		(start 129.54 99.06)
-		(end 129.54 100.192786)
-		(width 0.2)
-		(layer "In2.Cu")
-		(net 2)
-	)
-	(segment
-		(start 129.54 100.192786)
-		(end 131.748214 102.401)
-		(width 0.2)
-		(layer "In2.Cu")
-		(net 2)
-	)
-	(segment
 		(start 127 99.06)
 		(end 121.92 104.14)
@@
 	)
 	(segment
-		(start 131.748214 102.401)
-		(end 132.411786 102.401)
+		(start 135.822 100.262)
+		(end 141.038 100.262)
 		(width 0.2)
 		(layer "In2.Cu")
@@
 	)
 	(segment
-		(start 135.421 97.321)
-		(end 133.181 95.081)
-		(width 0.2)
-		(layer "In2.Cu")
-		(net 36)
-	)
-	(segment
 		(start 119.042 91.44)
 		(end 109.22 91.44)
@@
 	(segment
 		(start 133.181 95.081)
-		(end 122.683 95.081)
+		(end 129.54 95.081)
 		(width 0.2)
 		(layer "In2.Cu")
@@
 	)
 	(segment
-		(start 94.43605 102.701)
-		(end 96.52 100.61705)
+		(start 132.08 97.621)
+		(end 129.54 95.081)
 		(width 0.2)
 		(layer "In2.Cu")
@@
 	)
 	(segment
-		(start 132.08 101.6)
-		(end 133.819 99.861)
+		(start 129.54 95.081)
+		(end 122.683 95.081)
 		(width 0.2)
 		(layer "In2.Cu")
@@
 	)
 	(segment
-		(start 66.04 101.6)
-		(end 55.88 101.6)
+		(start 94.43605 102.701)
+		(end 96.52 100.61705)
 		(width 0.2)
 		(layer "In2.Cu")
@@
 	)
 	(segment
-		(start 109.22 91.44)
-		(end 106.68 88.9)
+		(start 66.04 101.6)
+		(end 55.88 101.6)
 		(width 0.2)
 		(layer "In2.Cu")
@@
 	)
 	(segment
-		(start 135.421 99.391786)
-		(end 135.421 97.321)
+		(start 109.22 91.44)
+		(end 106.68 88.9)
 		(width 0.2)
 		(layer "In2.Cu")
@@
 	)
 	(segment
-		(start 134.951786 99.861)
-		(end 135.421 99.391786)
-		(width 0.2)
-		(layer "In2.Cu")
-		(net 36)
-	)
-	(segment
 		(start 96.52 93.98)
 		(end 101.6 88.9)
@@
 	)
 	(segment
-		(start 133.819 99.861)
-		(end 134.951786 99.861)
+		(start 132.08 101.6)
+		(end 132.08 97.621)
 		(width 0.2)
 		(layer "In2.Cu")
@@
 	)
 	(segment
-		(start 134.62 99.06)
-		(end 134.62 101.6)
+		(start 76.2 104.14)
+		(end 76.2 116.84)
 		(width 1.5)
 		(layer "B.Cu")
@@
 	)
 	(segment
-		(start 76.2 104.14)
-		(end 76.2 116.84)
+		(start 129.54 99.06)
+		(end 129.54 101.6)
 		(width 1.5)
 		(layer "B.Cu")
@@
 	)
 	(segment
-		(start 138.261 117.941)
-		(end 138.261 107.781)
+		(start 122.46 96.52)
+		(end 123.561 97.621)
 		(width 0.2)
 		(layer "In2.Cu")
@@
 	)
 	(segment
-		(start 142.24 121.92)
-		(end 138.261 117.941)
+		(start 122.46 98.52)
+		(end 116.84 104.14)
 		(width 0.2)
 		(layer "In2.Cu")
@@
 	)
 	(segment
-		(start 122.46 96.52)
-		(end 123.561 97.621)
+		(start 129.54 101.6)
+		(end 132.08 104.14)
 		(width 0.2)
 		(layer "In2.Cu")
@@
 	)
 	(segment
-		(start 122.46 98.52)
-		(end 116.84 104.14)
+		(start 99.06 104.14)
+		(end 88.9 104.14)
 		(width 0.2)
 		(layer "In2.Cu")
@@
 	)
 	(segment
-		(start 123.561 97.621)
-		(end 133.181 97.621)
+		(start 122.46 96.52)
+		(end 122.46 98.52)
 		(width 0.2)
 		(layer "In2.Cu")
@@
 	)
 	(segment
-		(start 133.181 97.621)
-		(end 134.62 99.06)
+		(start 129.54 99.06)
+		(end 128.101 97.621)
 		(width 0.2)
 		(layer "In2.Cu")
@@
 	)
 	(segment
-		(start 134.62 104.14)
-		(end 138.261 107.781)
+		(start 138.261 117.941)
+		(end 142.24 121.92)
 		(width 0.2)
 		(layer "In2.Cu")
@@
 	)
 	(segment
-		(start 134.62 101.6)
-		(end 134.62 104.14)
+		(start 128.101 97.621)
+		(end 123.561 97.621)
 		(width 0.2)
 		(layer "In2.Cu")
@@
 	)
 	(segment
-		(start 99.06 104.14)
-		(end 88.9 104.14)
+		(start 134.62 104.14)
+		(end 138.261 107.781)
 		(width 0.2)
 		(layer "In2.Cu")
@@
 	)
 	(segment
-		(start 122.46 96.52)
-		(end 122.46 98.52)
+		(start 138.261 107.781)
+		(end 138.261 117.941)
+		(width 0.2)
+		(layer "In2.Cu")
+		(net 40)
+	)
+	(segment
+		(start 132.08 104.14)
+		(end 134.62 104.14)
 		(width 0.2)
 		(layer "In2.Cu")
